File: FRAM mini-shield/FRAM-mini-shield.kicad_pcb (KiCad board)
At the start: 2 copper layers, 24.9 x 53.3 mm, 30 parts, among them U1 MB85RS1MT, U2 MB85RS1MT, U3 MB85RS1MT, U4 TXB0108

Commit message: 2014-11-05 release.
Parts:
- removed the G*** at (123.8, 157.7)
- removed JMP1: 5V, ab2_header:AB2_SJMP_02-1
- removed JMP2: 3.3V, ab2_header:AB2_SJMP_02-1
- removed JMP3: SCK, ab2_header:AB2_SJMP_02-1
- removed JMP4: MISO, ab2_header:AB2_SJMP_02-1
- removed JMP5: MOSI, ab2_header:AB2_SJMP_02-1
- removed JMP6: CSU3, ab2_header:AB2_SJMP_02-1
- removed JMP7: CSU2, ab2_header:AB2_SJMP_02-1
- removed JMP8: CSU1, ab2_header:AB2_SJMP_02-1
- added G***: LOGO, Hackscribble_Logo:logo-small, F.Cu at (124.3, 159.3)
- HDR1: value AB2_HDR05-1 -> AB2_HDR08-1; footprint ab2_header:AB2_HDR_M05-1V -> ab2_header:AB2_HDR_M08-1V
- HDR7: value CSU3 -> D10-U3
- HDR8: value CSU2 -> D9-U2
- HDR9: value CSU1 -> D8-U1
- moved HDR1 3.81 mm to (122.2, 175.3)
Connections:
- C1 pad 1: Net-(C1-Pad1) -> +3.3V
- C2 pad 1: Net-(C1-Pad1) -> +3.3V
- C3 pad 1: Net-(C1-Pad1) -> +3.3V
- C4 pad 1: Net-(C1-Pad1) -> +3.3V
- C5 pad 1: Net-(C1-Pad1) -> +3.3V
- C6 pad 1: Net-(C1-Pad1) -> +3.3V
- C7 pad 1: +5V -> Net-(C7-Pad1)
- HDR1 pad 4: +5V -> Net-(HDR1-Pad4)
- U1 pad 3: Net-(C1-Pad1) -> +3.3V
- U1 pad 7: Net-(C1-Pad1) -> +3.3V
- U1 pad 8: Net-(C1-Pad1) -> +3.3V
- U2 pad 3: Net-(C1-Pad1) -> +3.3V
- U2 pad 7: Net-(C1-Pad1) -> +3.3V
- U2 pad 8: Net-(C1-Pad1) -> +3.3V
- U3 pad 3: Net-(C1-Pad1) -> +3.3V
- U3 pad 7: Net-(C1-Pad1) -> +3.3V
- U3 pad 8: Net-(C1-Pad1) -> +3.3V
- U4 pad 19: +5V -> Net-(C7-Pad1)
Routing:
- net Net-(C1-Pad1): track 72.5 -> 0.00 mm, vias 5 -> 0
- net +5V: track 65.0 -> 0.00 mm, vias 1 -> 0
- net +3.3V: track 65.7 -> 122.5 mm, vias 1 -> 4
- net Net-(C7-Pad1): track 0.00 -> 55.3 mm, vias 0 -> 1
- net Net-(HDR2-Pad5): track 26.7 -> 4.03 mm
- net Net-(HDR2-Pad4): track 23.6 -> 3.17 mm
- net Net-(HDR2-Pad3): track 21.8 -> 3.73 mm
- net Net-(HDR2-Pad2): track 21.6 -> 5.53 mm
- net Net-(HDR2-Pad1): track 22.0 -> 7.05 mm
- net Net-(HDR2-Pad6): track 20.3 -> 5.82 mm, vias 1 -> 0
- net Net-(HDR7-Pad1): track 80.0 -> 65.9 mm
- net Net-(HDR4-Pad1): track 65.2 -> 59.3 mm
- net Net-(HDR9-Pad1): track 41.1 -> 36.2 mm
- net Net-(HDR6-Pad1): track 49.0 -> 46.0 mm
- net Net-(HDR5-Pad1): track 63.0 -> 61.5 mm, vias 5 -> 4
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Other:
- outline, holes or cut-outs redrawn
- board text added: "REVISION B"
- board text added: "Use 3.3V FRAMs"
- board text removed: "REVISION A"
